Commit message: Gazebo now properly display the robot. Collision and Moveit are not working

File: src/CLOVIS25_URDF_Assembly_V1/urdf/CLOVIS25_URDF_Assembly_V1.urdf (robot description, URDF)
Before this commit: robot CLOVIS25_URDF_Assembly_V1, 18 links, 17 joints
Links:
- link Link10_AxisRy_Hips_Flexion: geometry collision mesh filename=file:///home/gmingant/CLOVIS-2-MINI-ROS2-Sim/src/CLOVIS25_U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; visual mesh filename=file:///home/gmingant/CLOVIS-2-MINI-ROS2-Sim/src/CLOVIS25_U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
- link Link11_AxisRx_Hips_Abduction: geometry collision mesh filename=file:///home/gmingant/CLOVIS-2-MINI-ROS2-Sim/src/CLOVIS25_U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; visual mesh filename=file:///home/gmingant/CLOVIS-2-MINI-ROS2-Sim/src/CLOVIS25_U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
- link Link12_AxisRz_Hips_Rotation: geometry collision mesh filename=file:///home/gmingant/CLOVIS-2-MINI-ROS2-Sim/src/CLOVIS25_U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; visual mesh filename=file:///home/gmingant/CLOVIS-2-MINI-ROS2-Sim/src/CLOVIS25_U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
- link Link13_AxisRy_Knee_Flexion: geometry collision mesh filename=file:///home/gmingant/CLOVIS-2-MINI-ROS2-Sim/src/CLOVIS25_U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; visual mesh filename=file:///home/gmingant/CLOVIS-2-MINI-ROS2-Sim/src/CLOVIS25_U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
- link Link14_AxisRy_Ankle_Flexion: geometry collision mesh filename=file:///home/gmingant/CLOVIS-2-MINI-ROS2-Sim/src/CLOVIS25_U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; visual mesh filename=file:///home/gmingant/CLOVIS-2-MINI-ROS2-Sim/src/CLOVIS25_U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
- link Link15_AxisRx_Ankle_Abduction: geometry collision mesh filename=file:///home/gmingant/CLOVIS-2-MINI-ROS2-Sim/src/CLOVIS25_U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; visual mesh filename=file:///home/gmingant/CLOVIS-2-MINI-ROS2-Sim/src/CLOVIS25_U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
- link Link16_AxisRx_Toe_Flexion: geometry collision mesh filename=file:///home/gmingant/CLOVIS-2-MINI-ROS2-Sim/src/CLOVIS25_U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; visual mesh filename=file:///home/gmingant/CLOVIS-2-MINI-ROS2-Sim/src/CLOVIS25_U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
- link Link1_AxisRx_Waist_Roll: geometry collision mesh filename=file:///home/gmingant/CLOVIS-2-MINI-ROS2-Sim/src/CLOVIS25_U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; visual mesh filename=file:///home/gmingant/CLOVIS-2-MINI-ROS2-Sim/src/CLOVIS25_U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
- link Link20_AxisRy_Hips_Flexion: geometry collision mesh filename=file:///home/gmingant/CLOVIS-2-MINI-ROS2-Sim/src/CLOVIS25_U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; visual mesh filename=file:///home/gmingant/CLOVIS-2-MINI-ROS2-Sim/src/CLOVIS25_U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
- link Link21_AxisRx_Hips_Abduction: geometry collision mesh filename=file:///home/gmingant/CLOVIS-2-MINI-ROS2-Sim/src/CLOVIS25_U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; visual mesh filename=file:///home/gmingant/CLOVIS-2-MINI-ROS2-Sim/src/CLOVIS25_U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
- link Link22_AxisRz_Hips_Rotation: geometry collision mesh filename=file:///home/gmingant/CLOVIS-2-MINI-ROS2-Sim/src/CLOVIS25_U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; visual mesh filename=file:///home/gmingant/CLOVIS-2-MINI-ROS2-Sim/src/CLOVIS25_U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
- link Link23_AxisRy_Knee_Flexion: geometry collision mesh filename=file:///home/gmingant/CLOVIS-2-MINI-ROS2-Sim/src/CLOVIS25_U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; visual mesh filename=file:///home/gmingant/CLOVIS-2-MINI-ROS2-Sim/src/CLOVIS25_U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
- link Link24_AxisRy_Ankle_Flexion: geometry collision mesh filename=file:///home/gmingant/CLOVIS-2-MINI-ROS2-Sim/src/CLOVIS25_U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; visual mesh filename=file:///home/gmingant/CLOVIS-2-MINI-ROS2-Sim/src/CLOVIS25_U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
- link Link25_AxisRx_Ankle_Abduction: geometry collision mesh filename=file:///home/gmingant/CLOVIS-2-MINI-ROS2-Sim/src/CLOVIS25_U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; visual mesh filename=file:///home/gmingant/CLOVIS-2-MINI-ROS2-Sim/src/CLOVIS25_U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
- link Link26_AxisRx_Toe_Flexion: geometry collision mesh filename=file:///home/gmingant/CLOVIS-2-MINI-ROS2-Sim/src/CLOVIS25_U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; visual mesh filename=file:///home/gmingant/CLOVIS-2-MINI-ROS2-Sim/src/CLOVIS25_U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
- link Link2_AxisRy_Abs_Pitch: geometry collision mesh filename=file:///home/gmingant/CLOVIS-2-MINI-ROS2-Sim/src/CLOVIS25_U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; visual mesh filename=file:///home/gmingant/CLOVIS-2-MINI-ROS2-Sim/src/CLOVIS25_U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
- link LinkR0_AxisRz_Waist_Yaw: geometry collision mesh filename=file:///home/gmingant/CLOVIS-2-MINI-ROS2-Sim/src/CLOVIS25_U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; visual mesh filename=file:///home/gmingant/CLOVIS-2-MINI-ROS2-Sim/src/CLOVIS25_U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
- link base_link_R0_HipsWaist_Yaw: geometry collision mesh filename=file:///home/gmingant/CLOVIS-2-MINI-ROS2-Sim/src/CLOVIS25_U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; visual mesh filename=file:///home/gmingant/CLOVIS-2-MINI-ROS2-Sim/src/CLOVIS25_U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

File: src/CLOVIS25_URDF_Assembly_V1_With_Arms/urdf/CLOVIS25_URDF_Assembly_V1 With Arms.urdf (robot description, URDF)
Before this commit: robot CLOVIS25_URDF_Assembly_V1 With Arms, 30 links, 29 joints
Links:
- link Link10_AxisRy_Hips_Flexion: geometry collision mesh filename=file:///home/gmingant/CLOVIS-2-MINI-ROS2-Sim/src/CLOVIS25_U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; visual mesh filename=file:///home/gmingant/CLOVIS-2-MINI-ROS2-Sim/src/CLOVIS25_U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
- link Link11_AxisRx_Hips_Abduction: geometry collision mesh filename=file:///home/gmingant/CLOVIS-2-MINI-ROS2-Sim/src/CLOVIS25_U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; visual mesh filename=file:///home/gmingant/CLOVIS-2-MINI-ROS2-Sim/src/CLOVIS25_U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
- link Link12_AxisRz_Hips_Rotation: geometry collision mesh filename=file:///home/gmingant/CLOVIS-2-MINI-ROS2-Sim/src/CLOVIS25_U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; visual mesh filename=file:///home/gmingant/CLOVIS-2-MINI-ROS2-Sim/src/CLOVIS25_U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
- link Link13_AxisRy_Knee_Flexion: geometry collision mesh filename=file:///home/gmingant/CLOVIS-2-MINI-ROS2-Sim/src/CLOVIS25_U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; visual mesh filename=file:///home/gmingant/CLOVIS-2-MINI-ROS2-Sim/src/CLOVIS25_U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
- link Link14_AxisRy_Ankle_Flexion: geometry collision mesh filename=file:///home/gmingant/CLOVIS-2-MINI-ROS2-Sim/src/CLOVIS25_U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; visual mesh filename=file:///home/gmingant/CLOVIS-2-MINI-ROS2-Sim/src/CLOVIS25_U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
- link Link15_AxisRx_Ankle_Abduction: geometry collision mesh filename=file:///home/gmingant/CLOVIS-2-MINI-ROS2-Sim/src/CLOVIS25_U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; visual mesh filename=file:///home/gmingant/CLOVIS-2-MINI-ROS2-Sim/src/CLOVIS25_U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
- link Link16_AxisRx_Toe_Flexion: geometry collision mesh filename=file:///home/gmingant/CLOVIS-2-MINI-ROS2-Sim/src/CLOVIS25_U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; visual mesh filename=file:///home/gmingant/CLOVIS-2-MINI-ROS2-Sim/src/CLOVIS25_U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
- link Link1_AxisRx_Abs_Roll: geometry collision mesh filename=file:///home/gmingant/CLOVIS-2-MINI-ROS2-Sim/src/CLOVIS25_U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; visual mesh filename=file:///home/gmingant/CLOVIS-2-MINI-ROS2-Sim/src/CLOVIS25_U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
- link Link20_AxisRy_Hips_Flexion: geometry collision mesh filename=file:///home/gmingant/CLOVIS-2-MINI-ROS2-Sim/src/CLOVIS25_U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; visual mesh filename=file:///home/gmingant/CLOVIS-2-MINI-ROS2-Sim/src/CLOVIS25_U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
- link Link21_AxisRx_Hips_Abduction: geometry collision mesh filename=file:///home/gmingant/CLOVIS-2-MINI-ROS2-Sim/src/CLOVIS25_U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; visual mesh filename=file:///home/gmingant/CLOVIS-2-MINI-ROS2-Sim/src/CLOVIS25_U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
- link Link22_AxisRz_Hips_Rotation: geometry collision mesh filename=file:///home/gmingant/CLOVIS-2-MINI-ROS2-Sim/src/CLOVIS25_U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; visual mesh filename=file:///home/gmingant/CLOVIS-2-MINI-ROS2-Sim/src/CLOVIS25_U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
- link Link23_AxisRy_Knee_Flexion: geometry collision mesh filename=file:///home/gmingant/CLOVIS-2-MINI-ROS2-Sim/src/CLOVIS25_U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; visual mesh filename=file:///home/gmingant/CLOVIS-2-MINI-ROS2-Sim/src/CLOVIS25_U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
- link Link24_AxisRy_Ankle_Flexion: geometry collision mesh filename=file:///home/gmingant/CLOVIS-2-MINI-ROS2-Sim/src/CLOVIS25_U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; visual mesh filename=file:///home/gmingant/CLOVIS-2-MINI-ROS2-Sim/src/CLOVIS25_U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
- link Link25_AxisRx_Ankle_Abduction: geometry collision mesh filename=file:///home/gmingant/CLOVIS-2-MINI-ROS2-Sim/src/CLOVIS25_U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; visual mesh filename=file:///home/gmingant/CLOVIS-2-MINI-ROS2-Sim/src/CLOVIS25_U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
- link Link26_AxisRx_Toe_Flexion: geometry collision mesh filename=file:///home/gmingant/CLOVIS-2-MINI-ROS2-Sim/src/CLOVIS25_U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; visual mesh filename=file:///home/gmingant/CLOVIS-2-MINI-ROS2-Sim/src/CLOVIS25_U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
- link Link2_AxisRy_Abs_Pitch: geometry collision mesh filename=file:///home/gmingant/CLOVIS-2-MINI-ROS2-Sim/src/CLOVIS25_U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; visual mesh filename=file:///home/gmingant/CLOVIS-2-MINI-ROS2-Sim/src/CLOVIS25_U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
- link Link30_AxisRy_Shoulder_Flexion: geometry collision mesh filename=file:///home/gmingant/CLOVIS-2-MINI-ROS2-Sim/src/CLOVIS25_U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; visual mesh filename=file:///home/gmingant/CLOVIS-2-MINI-ROS2-Sim/src/CLOVIS25_U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
- link Link31_AxisRz_Shoulder_Rotation: geometry collision mesh filename=file:///home/gmingant/CLOVIS-2-MINI-ROS2-Sim/src/CLOVIS25_U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; visual mesh filename=file:///home/gmingant/CLOVIS-2-MINI-ROS2-Sim/src/CLOVIS25_U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
- link Link32_AxisRx_Shoulder_Abduction: geometry collision mesh filename=file:///home/gmingant/CLOVIS-2-MINI-ROS2-Sim/src/CLOVIS25_U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; visual mesh filename=file:///home/gmingant/CLOVIS-2-MINI-ROS2-Sim/src/CLOVIS25_U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
- link Link33_AxisRy_Elbow_Flexion: geometry collision mesh filename=file:///home/gmingant/CLOVIS-2-MINI-ROS2-Sim/src/CLOVIS25_U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; visual mesh filename=file:///home/gmingant/CLOVIS-2-MINI-ROS2-Sim/src/CLOVIS25_U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
- link Link34_AxisRz_Wrist_Rotation: geometry collision mesh filename=file:///home/gmingant/CLOVIS-2-MINI-ROS2-Sim/src/CLOVIS25_U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; visual mesh filename=file:///home/gmingant/CLOVIS-2-MINI-ROS2-Sim/src/CLOVIS25_U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
- link Link35_AxisRx_Wrist_Abduction: geometry collision mesh filename=file:///home/gmingant/CLOVIS-2-MINI-ROS2-Sim/src/CLOVIS25_U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; visual mesh filename=file:///home/gmingant/CLOVIS-2-MINI-ROS2-Sim/src/CLOVIS25_U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
- link Link40_AxisRy_Shoulder_Flexion: geometry collision mesh filename=file:///home/gmingant/CLOVIS-2-MINI-ROS2-Sim/src/CLOVIS25_U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; visual mesh filename=file:///home/gmingant/CLOVIS-2-MINI-ROS2-Sim/src/CLOVIS25_U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
- link Link41_AxisRz_Shoulder_Rotation: geometry collision mesh filename=file:///home/gmingant/CLOVIS-2-MINI-ROS2-Sim/src/CLOVIS25_U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; visual mesh filename=file:///home/gmingant/CLOVIS-2-MINI-ROS2-Sim/src/CLOVIS25_U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
- link Link42_AxisRx_Shoulder_Abduction: geometry collision mesh filename=file:///home/gmingant/CLOVIS-2-MINI-ROS2-Sim/src/CLOVIS25_U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; visual mesh filename=file:///home/gmingant/CLOVIS-2-MINI-ROS2-Sim/src/CLOVIS25_U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
- link Link43_AxisRy_Elbow_Flexion: geometry collision mesh filename=file:///home/gmingant/CLOVIS-2-MINI-ROS2-Sim/src/CLOVIS25_U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; visual mesh filename=file:///home/gmingant/CLOVIS-2-MINI-ROS2-Sim/src/CLOVIS25_U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
- link Link44_AxisRz_Wrist_Rotation: geometry collision mesh filename=file:///home/gmingant/CLOVIS-2-MINI-ROS2-Sim/src/CLOVIS25_U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; visual mesh filename=file:///home/gmingant/CLOVIS-2-MINI-ROS2-Sim/src/CLOVIS25_U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
- link Link45_AxisRx_Wrist_Abduction: geometry collision mesh filename=file:///home/gmingant/CLOVIS-2-MINI-ROS2-Sim/src/CLOVIS25_U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; visual mesh filename=file:///home/gmingant/CLOVIS-2-MINI-ROS2-Sim/src/CLOVIS25_U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
- link LinkR0_AxisRz_Waist_Yaw: geometry collision mesh filename=file:///home/gmingant/CLOVIS-2-MINI-ROS2-Sim/src/CLOVIS25_U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; visual mesh filename=file:///home/gmingant/CLOVIS-2-MINI-ROS2-Sim/src/CLOVIS25_U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
- link base_link_R0_HipsWaist_Yaw: geometry collision mesh filename=file:///home/gmingant/CLOVIS-2-MINI-ROS2-Sim/src/CLOVIS25_U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; visual mesh filename=file:///home/gmingant/CLOVIS-2-MINI-ROS2-Sim/src/CLOVIS25_U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

File: src/robot_description/urdf/clovis2mini.urdf.xacro (robot description, xacro)
@@ -1,1043 +1,1742 @@
 <?xml version="1.0" encoding="utf-8"?>
-  <robot name="CLOVIS2Mini" xmlns:xacro="http://www.ros.org/wiki/xacro">
-    <link name="world" />
-    <joint name="base_joint" type="fixed">
-      <origin xyz="0 0 0" rpy="0 0 0" />
-      <parent link="world" />
-      <child link="base_link" />
-    </joint>
-    <link name="base_link" />
-    <joint name="base_link_fixed" type="fixed">
-      <origin xyz="0 0 0" rpy="0 0 0" />
-      <parent link="base_link" />
-      <child link="base_link_R0_HipsWaist_Yaw" />
-    </joint>
-    <link
-  name="base_link_R0_HipsWaist_Yaw">
-  <inertial>
-    <origin
-      xyz="5.0364E-07 -0.0073562 0.0064621"
-      rpy="0 0 0" />
-    <mass
-      value="0.38744" />
-    <inertia
-      ixx="0.000602"
-      ixy="-8.4057E-09"
-      ixz="3.9044E-09"
-      iyy="0.00059139"
-      iyz="0.00014423"
-      izz="0.00055466" />
-  </inertial>
-  <visual>
+<robot name="CLOVIS2Mini" xmlns:xacro="http://www.ros.org/wiki/xacro">
+  <link name="world" />
+  <joint name="base_joint" type="fixed">
+    <origin xyz="0 0 0" rpy="0 0 0" />
+    <parent link="world" />
+    <child link="base_link" />
+  </joint>
+  <link name="base_link" />
+  <gazebo>
+    <self_collide>false</self_collide>
+  </gazebo>
+  <joint name="base_link_fixed" type="fixed">
+    <origin xyz="0 0 0" rpy="0 0 0" />
+    <parent link="base_link" />
+    <child link="base_link_R0_HipsWaist_Yaw" />
+  </joint>
+<link
+    name="base_link_R0_HipsWaist_Yaw">
+    <inertial>
+      <origin
+        xyz="-5.06849795022235E-07 0.00646210878121357 -0.0073561947767718"
+        rpy="0 0 0" />
+      <mass
+        value="0.387437520077023" />
+      <inertia
+        ixx="0.000602004181055371"
+        ixy="-3.93523733518146E-09"
+        ixz="8.41311460772213E-09"
+        iyy="0.000554663199182993"
+        iyz="0.000144231027666502"
+        izz="0.000591393422247619" />
+    </inertial>
+    <visual>
+      <origin
+        xyz="0 0 0"
+        rpy="0 0 0" />
+      <geometry>
+        <mesh
+          filename="file:///home/gmingant/CLOVIS-2-MINI-ROS2-Sim/src/CLOVIS25_URDF_Assembly_V1_With_Arms/meshes/base_link_R0_HipsWaist_Yaw.STL" />
+      </geometry>
+      <material
+        name="">
+        <color
+          rgba="0.752941176470588 0.752941176470588 0.752941176470588 1" />
+      </material>
+    </visual>
+    <collision>
+      <origin
+        xyz="0 0 0"
+        rpy="0 0 0" />
+      <geometry>
+        <mesh
+          filename="file:///home/gmingant/CLOVIS-2-MINI-ROS2-Sim/src/CLOVIS25_URDF_Assembly_V1_With_Arms/meshes/base_link_R0_HipsWaist_Yaw.STL" />
+      </geometry>
+    </collision>
+  </link>
+  <link
+    name="LinkR0_AxisRz_Waist_Yaw">
+    <inertial>
+      <origin
+        xyz="1.4681236456414E-08 0.00792255367963898 0.0328105533698632"
+        rpy="0 0 0" />
+      <mass
+        value="0.0743770113903965" />
+      <inertia
+        ixx="0.000109844902331301"
+        ixy="6.43572844053016E-11"
+        ixz="1.80691197728788E-11"
+        iyy="5.27744826789087E-05"
+        iyz="8.6681121560006E-06"
+        izz="6.86185978836166E-05" />
+    </inertial>
+    <visual>
+      <origin
+        xyz="0 0 0"
+        rpy="0 0 0" />
+      <geometry>
+        <mesh
+          filename="file:///home/gmingant/CLOVIS-2-MINI-ROS2-Sim/src/CLOVIS25_URDF_Assembly_V1_With_Arms/meshes/LinkR0_AxisRz_Waist_Yaw.STL" />
+      </geometry>
+      <material
+        name="">
+        <color
+          rgba="0.752941176470588 0.752941176470588 0.752941176470588 1" />
+      </material>
+    </visual>
+    <collision>
+      <origin
+        xyz="0 0 0"
+        rpy="0 0 0" />
+      <geometry>
+        <mesh
+          filename="file:///home/gmingant/CLOVIS-2-MINI-ROS2-Sim/src/CLOVIS25_URDF_Assembly_V1_With_Arms/meshes/LinkR0_AxisRz_Waist_Yaw.STL" />
+      </geometry>
+    </collision>
+  </link>
+  <joint
+    name="R0_AxisRz_Waist_Yaw"
+    type="revolute">
     <origin
       xyz="0 0 0"
       rpy="0 0 0" />
-    <geometry>
-      <mesh
-        filename="package://robot_description/meshes/base_link_R0_HipsWaist_Yaw.STL" />
-    </geometry>
-    <material
-      name="">
-      <color
-        rgba="0.75294 0.75294 0.75294 1" />
-    </material>
-  </visual>
-  <collision>
+    <parent
+      link="base_link_R0_HipsWaist_Yaw" />
+    <child
+      link="LinkR0_AxisRz_Waist_Yaw" />
+    <axis
+      xyz="0 0 1" />
+    <limit
+      lower="-0.611"
+      upper="0.611"
+      effort="3.66"
+      velocity="5.05" />
+  </joint>
+  <link
+    name="Link1_AxisRx_Abs_Roll">
+    <inertial>
+      <origin
+        xyz="-0.000419037666760606 -8.67044488973194E-06 0.00334728947605621"
+        rpy="0 0 0" />
+      <mass
+        value="0.0285702910432507" />
+      <inertia
+        ixx="7.08725803682833E-06"
+        ixy="-2.45830099310385E-09"
+        ixz="-4.77409616773028E-08"
+        iyy="2.32521875946385E-05"
+        iyz="-1.5933209297635E-09"
+        izz="2.62164733137173E-05" />
+    </inertial>
+    <visual>
+      <origin
+        xyz="0 0 0"
+        rpy="0 0 0" />
+      <geometry>
+        <mesh
+          filename="file:///home/gmingant/CLOVIS-2-MINI-ROS2-Sim/src/CLOVIS25_URDF_Assembly_V1_With_Arms/meshes/Link1_AxisRx_Abs_Roll.STL" />
+      </geometry>
+      <material
+        name="">
+        <color
+          rgba="0.698039215686274 0.698039215686274 0.698039215686274 1" />
+      </material>
+    </visual>
+    <collision>
+      <origin
+        xyz="0 0 0"
+        rpy="0 0 0" />
+      <geometry>
+        <mesh
+          filename="file:///home/gmingant/CLOVIS-2-MINI-ROS2-Sim/src/CLOVIS25_URDF_Assembly_V1_With_Arms/meshes/Link1_AxisRx_Abs_Roll.STL" />
+      </geometry>
+    </collision>
+  </link>
+  <joint
+    name="R1_AxisRx_Abs_Roll"
+    type="revolute">
+    <origin
+      xyz="0 0 0.0830000000000002"
+      rpy="0 0 1.5707963267949" />
+    <parent
+      link="LinkR0_AxisRz_Waist_Yaw" />
+    <child
+      link="Link1_AxisRx_Abs_Roll" />
+    <axis
+      xyz="-1 0 0" />
+    <limit
+      lower="-0.524"
+      upper="0.524"
+      effort="3.66"
+      velocity="5.05" />
+  </joint>
+  <link
+    name="Link2_AxisRy_Abs_Pitch">
+    <inertial>
+      <origin
+        xyz="0.011650181340946 0.000444755928511933 0.099005739309927"
+        rpy="0 0 0" />
+      <mass
+        value="1.76578959011334" />
+      <inertia
+        ixx="0.00272833770431028"
+        ixy="-2.20264076877396E-07"
+        ixz="8.18791936776388E-05"
+        iyy="0.00286417266365648"
+        iyz="4.10696306321673E-07"
+        izz="0.00262213376829883" />
+    </inertial>
+    <visual>
+      <origin
+        xyz="0 0 0"
+        rpy="0 0 0" />
+      <geometry>
+        <mesh
+          filename="file:///home/gmingant/CLOVIS-2-MINI-ROS2-Sim/src/CLOVIS25_URDF_Assembly_V1_With_Arms/meshes/Link2_AxisRy_Abs_Pitch.STL" />
+      </geometry>
+      <material
+        name="">
+        <color
+          rgba="0.752941176470588 0.752941176470588 0.752941176470588 1" />
+      </material>
+    </visual>
+    <collision>
+      <origin
+        xyz="0 0 0"
+        rpy="0 0 0" />
+      <geometry>
+        <mesh
+          filename="file:///home/gmingant/CLOVIS-2-MINI-ROS2-Sim/src/CLOVIS25_URDF_Assembly_V1_With_Arms/meshes/Link2_AxisRy_Abs_Pitch.STL" />
+      </geometry>
+    </collision>
+  </link>
+  <joint
+    name="R2_AxisRy_Abs_Pitch"
+    type="revolute">
     <origin
       xyz="0 0 0"
       rpy="0 0 0" />
-    <geometry>
-      <mesh
-        filename="package://robot_description/meshes/base_link_R0_HipsWaist_Yaw.STL" />
-    </geometry>
-  </collision>
-</link>
-<link
-  name="LinkR0_AxisRz_Waist_Yaw">
-  <inertial>
-    <origin
-      xyz="0.0079226 -1.4681E-08 0.032811"
+    <parent
+      link="Link1_AxisRx_Abs_Roll" />
+    <child
+      link="Link2_AxisRy_Abs_Pitch" />
+    <axis
+      xyz="0 -1 0" />
+    <limit
+      lower="-0.689"
+      upper="0.785"
+      effort="3.66"
+      velocity="5.05" />
+  </joint>
+  <link
+    name="Link30_AxisRy_Shoulder_Flexion">
+    <inertial>
+      <origin
+        xyz="-0.00121122065822793 -0.00325038076073686 0.0120544903508707"
+        rpy="0 0 0" />
+      <mass
+        value="0.037258013070383" />
+      <inertia
+        ixx="1.59289941290387E-05"
+        ixy="-1.20792452999147E-06"
+        ixz="-4.79405065236246E-07"
+        iyy="1.63933970089758E-05"
+        iyz="-8.02786738789969E-07"
+        izz="2.03149647590168E-05" />
+    </inertial>
+    <visual>
+      <origin
+        xyz="0 0 0"
+        rpy="0 0 0" />
+      <geometry>
+        <mesh
+          filename="file:///home/gmingant/CLOVIS-2-MINI-ROS2-Sim/src/CLOVIS25_URDF_Assembly_V1_With_Arms/meshes/Link30_AxisRy_Shoulder_Flexion.STL" />
+      </geometry>
+      <material
+        name="">
+        <color
+          rgba="0.752941176470588 0.752941176470588 0.752941176470588 1" />
+      </material>
+    </visual>
+    <collision>
+      <origin
+        xyz="0 0 0"
+        rpy="0 0 0" />
+      <geometry>
+        <mesh
+          filename="file:///home/gmingant/CLOVIS-2-MINI-ROS2-Sim/src/CLOVIS25_URDF_Assembly_V1_With_Arms/meshes/Link30_AxisRy_Shoulder_Flexion.STL" />
+      </geometry>
+    </collision>
+  </link>
+  <joint
+    name="R30_AxisRy_Shoulder_Flexion"
+    type="revolute">
+    <origin
+      xyz="0.028926 -0.10137 0.13085"
+      rpy="-0.25268 1.3002 -1.5708" />
+    <parent
+      link="Link2_AxisRy_Abs_Pitch" />
+    <child
+      link="Link30_AxisRy_Shoulder_Flexion" />
+    <axis
+      xyz="0 0 1" />
+    <limit
+      lower="0"
+      upper="0"
+      effort="0"
+      velocity="0" />
+  </joint>
+  <link
+    name="Link31_AxisRz_Shoulder_Rotation">
+    <inertial>
+      <origin
+        xyz="0.0310376632963731 0.0149615998455133 -0.00284843103933194"
+        rpy="0 0 0" />
+      <mass
+        value="0.0306387760752887" />
+      <inertia
+        ixx="1.91180450287481E-05"
+        ixy="-2.81655737035407E-07"
+        ixz="8.4332813770904E-07"
+        iyy="2.6492735208956E-05"
+        iyz="-1.49756484162903E-07"
+        izz="1.4496990488765E-05" />
+    </inertial>
+    <visual>
+      <origin
+        xyz="0 0 0"
+        rpy="0 0 0" />
+      <geometry>
+        <mesh
+          filename="file:///home/gmingant/CLOVIS-2-MINI-ROS2-Sim/src/CLOVIS25_URDF_Assembly_V1_With_Arms/meshes/Link31_AxisRz_Shoulder_Rotation.STL" />
+      </geometry>
+      <material
+        name="">
+        <color
+          rgba="0.752941176470588 0.752941176470588 0.752941176470588 1" />
+      </material>
+    </visual>
+    <collision>
+      <origin
+        xyz="0 0 0"
+        rpy="0 0 0" />
+      <geometry>
+        <mesh
+          filename="file:///home/gmingant/CLOVIS-2-MINI-ROS2-Sim/src/CLOVIS25_URDF_Assembly_V1_With_Arms/meshes/Link31_AxisRz_Shoulder_Rotation.STL" />
+      </geometry>
+    </collision>
+  </link>
+  <joint
+    name="R31_AxisRz_Shoulder_Rotation"
+    type="revolute">
+    <origin
+      xyz="0 0 0.0185"
+      rpy="1.5708 -1.3181 -1.5708" />
+    <parent
+      link="Link30_AxisRy_Shoulder_Flexion" />
+    <child
+      link="Link31_AxisRz_Shoulder_Rotation" />
+    <axis
+      xyz="0 0 -1" />
+    <limit
+      lower="0"
+      upper="0"
+      effort="0"
+      velocity="0" />
+  </joint>
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