Commit message: URDF hands fix (right thumb remain to be fix), limits remain to be add

File: src/CLOVIS25_URDF_V1/urdf/CLOVIS25_URDF_V1.urdf (robot description, URDF)
Before this commit: robot CLOVIS25_URDF_V1, 58 links, 57 joints
Links:
- link Link16_AxisRx_Toe_Flexion: mass 0.0664189830579756 -> 0.0664189830579757
- link Link20_AxisRy_Hips_Flexion: mass 0.150034857109824 -> 0.150034857109825
- link Link23_AxisRy_Knee_Flexion: mass 0.208100936749785 -> 0.208100936749786
- link Link25_AxisRx_Ankle_Abduction: mass 0.162069791661843 -> 0.162069791661844
- link Link33_AxisRy_Elbow_Flexion: mass 0.0625251373156171 -> 0.062525137315617
- link Link36_AxisRy_Wrist_Flexion: mass 0.094866835573617 -> 0.0948668355736169
- link Link40_AxisRy_Shoulder_Flexion: mass 0.0372585040292267 -> 0.0372585040292266
- link Link44_AxisRz_Wrist_Rotation: mass 0.0957043837946211 -> 0.0957043837946212
- link Link61_AxisRz_ThumbKnucle_Rotation: mass 0.00115968038152585 -> 0.00115968038152584
- link LinkR0_AxisRz_Waist_Yaw: mass 0.0743770113903967 -> 0.0743770113903965
- link base_link_R0_HipsWaist_Yaw: mass 0.387437520077023 -> 0.387437520077022
Joints:
- joint R35_AxisRx_Wrist_Abduction: axis 0 0 -1 -> 0 0 1; origin xyz=0 0 -0.0931377805455123 rpy=3.14159265358979 -1.5707963267949 0 -> xyz=0 0 -0.0931377805455123 rpy=0 1.5707963267949 0
- joint R36_AxisRy_Wrist_Flexion: axis 0 0 -1 -> 0 0 1; origin xyz=0 0 0 rpy=1.5707963267949 -1.48352986419518 0 -> xyz=0 0 0 rpy=-1.5707963267949 -1.48352986419518 0
- joint R51_AxisRz_ThumbKnucle_Rotation: origin xyz=0.0208992160414317 0.0382 -0.0217863192850372 rpy=-1.5707963267949 0 3.14159265358979 -> xyz=-0.020899 0.0382 0.021786 rpy=1.5708 0 0
- joint R52_AxisRy_ThumbKnucle_Flexion: origin xyz=0 0.0289711683278987 -0.00778918517667555 rpy=3.14159265358979 -1.5707963267949 0 -> xyz=0 0.028971 -0.0077892 rpy=3.1416 -1.5708 0
- joint R54_AxisRx_IndexKnucle_Abduction: origin xyz=0 0.100710889132455 -0.0300000000000001 rpy=-1.5707963267949 0 -1.5707963267949 -> xyz=0 0.10071 0.03 rpy=1.5708 0 -1.5708
- joint R55_AxisRy_IndexKnucle_Flexion: origin xyz=0 0 0 rpy=1.5707963267949 -1.5707963267949 0 -> xyz=0 0 0 rpy=1.5708 -1.5708 0
- joint R58_AxisRy_MiddleFingerKnucle_Flexion: origin xyz=0 0.0957999999999998 -0.0121 rpy=0 0 0 -> xyz=0 0.0957999999999998 0.0121 rpy=3.14159265358979 0 -3.14159265358979
- joint R62_AxisRy_ThumbKnucle_Flexion: axis 0 0 -1 -> 0 0 1; origin xyz=0 0 0 rpy=3.14159265358979 -1.5707963267949 0 -> xyz=0 0 0 rpy=0 1.5707963267949 0
- joint R63_AxisRy_Thumb_Flexion: origin xyz=0.00778918517667519 0.0289711683278997 -9.9999999999989E-05 rpy=-3.14159265358979 0 3.14159265358979 -> xyz=-0.00778918517667519 0.0289711683278997 9.9999999999989E-05 rpy=0 0 0
- joint R65_AxisRy_IndexKnucle_Flexion: origin xyz=0 0 0 rpy=1.5707963267949 -1.5707963267949 0 -> xyz=0 0 0 rpy=1.57079632679489 1.5707963267949 0
- joint R66_AxisRy_IndexMiddle_Flexion: origin xyz=0 0.0300000000000014 -9.99999999971579E-05 rpy=3.14159265358979 0 -3.14159265358979 -> xyz=0 0.0300000000000014 9.99999999971579E-05 rpy=0 0 0
- joint R72_AxisRy_PinkyKnucle_Flexion: origin xyz=0 0.0957999999999998 0.0238999999999999 rpy=0 0 0 -> xyz=0 0.0957999999999998 -0.0238999999999999 rpy=3.14159265358979 0 -3.14159265358979
- joint R83_AxisRy_PinkyMiddle_Flexion: origin xyz=0 0.03 0.0179 rpy=-3.1416 0 3.1416 -> xyz=0 0.0299999999999947 0.0178999999999945 rpy=-3.14159265358979 0 3.14159265358979
- joint R84_AxisRy_PinkyTip_Flexion: origin xyz=-0.00093853 0.018977 -0.0001 rpy=0 0 0 -> xyz=-0.000938526804095008 0.0189768060388963 -9.99999999999994E-05 rpy=0 0 0
